Commit message: CODICE SISTEMATO CON NUOVE BAG

File: src/mapping/robot/wall-e.urdf (robot description, URDF)
Before this commit: robot wall-e, 1 links, 0 joints
Links:
- removed link base_link
- added link scout/base_link; visual mesh filename=package://mapping/mesh/Wall-E_Scaled.stl scale=0.01 0.01 0.01
